File: PCB/skyboard.kicad_pcb (KiCad board)
At the start: 2 copper layers, 60 x 62 mm, 10 parts, among them SW1 SW_Push, SW2 SW_Push, SW3 SW_Push, SW4 SW_Push, SW5 SW_Push, SW6 SW_Push, SW7 RotaryEncoder_Switch, U1 XIAO-RP2040-DIP

Commit message: Added extra LEDs under the switches, fixed wiring
Parts:
- added D3: SK6812MINI, Hackclub Footprints:MX_SK6812MINI-E_REV, F.Cu at (138.1, 109.5)
- added D4: SK6812MINI, Hackclub Footprints:MX_SK6812MINI-E_REV, F.Cu at (138.1, 128.6)
- added D5: SK6812MINI, Hackclub Footprints:MX_SK6812MINI-E_REV, F.Cu at (157.2, 128.6)
- added D6: SK6812MINI, Hackclub Footprints:MX_SK6812MINI-E_REV, F.Cu at (157.2, 109.5)
- D1, D2: footprint LED_SMD:LED_SK6812MINI_PLCC4_3.5x3.5mm_P1.75mm -> Hackclub Footprints:MX_SK6812MINI-E_REV
- U1: footprint OPL:XIAO-RP2040-DIP -> Hackclub Footprints:XIAO-RP2040-DIP
- moved D1 47.2 mm to (119.1, 128.6)
- moved D2 27.9 mm to (119.1, 109.5)
Connections:
- D1 pad 2: Net-(D1-VSS) -> GND
- D1 pad 4: Net-(D1-VDD) -> +5V
- D2 pad 1: unconnected-(D2-DOUT-Pad1) -> Net-(D2-DOUT)
- D2 pad 2: Net-(D1-VSS) -> GND
- D2 pad 4: Net-(D1-VDD) -> +5V
- SW7 pad C: Net-(D1-VSS) -> GND
- SW7 pad S2: unconnected-(SW7-PadS2) -> GND
Routing:
- net +5V: track 0.00 -> 161.0 mm, vias 0 -> 8
- net GND: track 168.7 -> 258.1 mm, vias 1 -> 3
- net Net-(D1-VSS): track 67.1 -> 0.00 mm, vias 1 -> 0
- net Net-(D1-DIN): track 21.9 -> 73.7 mm, vias 1 -> 0
- net Net-(D5-DOUT): track 0.00 -> 39.6 mm
- net Net-(D3-DOUT): track 0.00 -> 32.4 mm
- net Net-(D1-VDD): track 16.5 -> 0.00 mm
- net Net-(D1-DOUT): track 27.0 -> 42.2 mm
- net Net-(D4-DOUT): track 0.00 -> 14.5 mm, vias 0 -> 2
- net Net-(D2-DOUT): track 0.00 -> 14.5 mm
- net Net-(U1-GPIO0/TX): track 22.6 -> 16.1 mm
Other:
- board text removed: "SkyBoard"
